Commit message: A total new code which is a hybrid method of Depth point and tracker for creating of obstacles.

File: yahboom_rosmaster_description/urdf/sensors/rgbd_camera.urdf.xacro (robot description, xacro)
@@ -8,5 +8,5 @@
     mesh_file:='file://$(find yahboom_rosmaster_description)/meshes/intel_realsense/visual/d435.stl'
     xyz_offset:='0.105 0 0.05'
-    rpy_offset:='0 -0.50 0'
+    rpy_offset:='0 0.2 0'
     mesh_xyz_offset:='0 0 0'
     mesh_rpy_offset:='${M_PI/2} 0.0 ${M_PI/2}'
@@ -41,5 +41,5 @@
     image_height:=240
     clip_near:=0.05
-    clip_far:=8.0
+    clip_far:=12.0
     update_rate:=5.0
     always_on:=1
@@ -49,17 +49,11 @@
       <visual>
         <origin xyz="${mesh_xyz_offset}" rpy="${mesh_rpy_offset}"/>
-        <geometry>
-          <mesh filename="${mesh_file}" />
-        </geometry>
-        <material name="${material_name}">
-          <color rgba="${material_color}"/>
-        </material>
+        <geometry><mesh filename="${mesh_file}" /></geometry>
+        <material name="${material_name}"><color rgba="${material_color}"/></material>
       </visual>
       <xacro:if value="${enable_collision}">
         <collision>
           <origin xyz="${collision_xyz_offset}" rpy="${collision_rpy_offset}"/>
-          <geometry>
-            <box size="${cam_depth} ${cam_width} ${cam_height}"/>
-          </geometry>
+          <geometry><box size="${cam_depth} ${cam_width} ${cam_height}"/></geometry>
         </collision>
       </xacro:if>
@@ -67,6 +61,5 @@
         <mass value="${mass}" />
         <origin xyz="${inertial_xyz_offset}" rpy="${inertial_rpy_offset}"/>
-        <inertia ixx="${ixx}" ixy="${ixy}" ixz="${ixz}"
-                 iyy="${iyy}" iyz="${iyz}" izz="${izz}" />
+        <inertia ixx="${ixx}" ixy="${ixy}" ixz="${ixz}" iyy="${iyy}" iyz="${iyz}" izz="${izz}" />
       </inertial>
     </link>
